File: ym2149.kicad_pcb (KiCad board)
At the start: 2 copper layers, 98.8 x 98.8 mm, 63 parts, among them J1 595_OUT, J10 UART, J11 I2C, J12 L GND R, J13 YM1_OUT, J14 GND, J15 YM2_OUT, J16 VCC, J17 OUT, J2 EXT_PWR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

Commit message: Add files via upload
Parts:
- JP1: value TCXO_EN -> CXO_EN
- X1: value TCXO-14 -> CXO-14
- moved J10 18.1 mm to (51.8, 78.7)
- moved C11 6.63 mm to (57.1, 94.4), turned to 90 degrees
- moved R12 6.07 mm to (59.8, 102.6), turned to 180 degrees
- moved C9 5.72 mm to (57.1, 82.0), turned to -90 degrees
- moved J11 3.98 mm to (51.8, 95.0)
- moved R11 3.42 mm to (59.8, 100.1), turned to 180 degrees
- moved D1 2.79 mm to (127.8, 38.1)
- moved D2 2.79 mm to (133.1, 38.1)
- moved R1 1.91 mm to (127.8, 41.3)
- moved R2 1.91 mm to (133.1, 41.3)
Connections:
- U2 pad 1: 595_RCLK -> 595_~{SRCLR}
- U2 pad 16: YM1_SEL -> YM1_BC1
- U2 pad 18: YM1_BC1 -> YM1_SEL
- U2 pad 4: 595_~{SRCLR} -> 595_RCLK
Routing:
- net 595_~{SRCLR}: track 24.7 -> 12.3 mm
- net YM1_BC1: track 57.7 -> 67.4 mm
- net 595_RCLK: track 10.5 -> 19.0 mm
- net SCL: track 27.0 -> 33.2 mm
- net YM1_SEL: track 56.7 -> 61.7 mm
- net TXD: track 23.8 -> 19.0 mm
- net SCK: track 86.1 -> 89.0 mm
- net SDA: track 29.4 -> 32.2 mm
- net RST: track 189.3 -> 191.2 mm
- net RXD: track 23.4 -> 21.7 mm
- net VCC: track 461.5 -> 462.5 mm
- net /XTAL2: track 9.00 -> 9.96 mm
- net Net-(D2-Pad1): track 2.28 -> 3.17 mm
- net Net-(D1-Pad1): track 2.28 -> 3.17 mm
- net GND: vias 57 -> 56
Other:
- board text added: "Dual YM2149 Synth REV. 2"
- board text removed: "Dual YM2149 Synth REV. 1a"
