File: ym2149.kicad_sch (KiCad schematic)
At the start: 59 parts, among them J1 595_OUT, J10 UART, J11 I2C, J12 L GND R, J13 YM1_OUT, J14 GND, J15 YM2_OUT, J16 VCC, J17 OUT, J2 EXT_PWR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

Commit message: Add files via upload
Parts:
- JP1: value TCXO_EN -> CXO_EN
- X1: value TCXO-14 -> CXO-14
Connections:
- net 595_RCLK: now also U2.4 (PB3); no longer U2.1 (PB0)
- net 595_~{SRCLR}: now also U2.1 (PB0); no longer U2.4 (PB3)
- net YM1_BC1: now also U2.16 (PD2); no longer U2.18 (PD4)
- net YM1_SEL: now also U2.18 (PD4); no longer U2.16 (PD2)
Other:
- company: (none) -> derleta.com
- title: (none) -> YM2149 Dual Synth
- moved on the sheet: C13, C4, F1, F2, J12, J13, J14, J15, J16, J17, J2, J3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
